File: Valkyre_Renew2.0.kicad_pcb (KiCad board)
At the start: 2 copper layers, 35.5 x 43 mm, 55 parts, among them J1 SWD, J16 TFT/OLED, J2 CAN2, J3 CAN2, J4 UART1, J5 UART3, J6 CAN1, J7 CAN1, SW2 RESET, SW3 BTN1, U1 TJA1050, U2 STM32F405RGTx, U3 TJA1050, U4 LP5907MFX-3.3, Y1 8.00MHz

Commit message: Add files via upload
Parts:
- R9: moved to F.Cu
- moved D3 41.2 mm to (178.5, 67.7), turned to -45 degrees
- moved D4 37.6 mm to (177.3, 68.9), turned to -45 degrees
- moved R9 32.2 mm to (179.0, 71.8), turned to 135 degrees
- moved D5 27.1 mm to (176.0, 70.1), turned to -45 degrees
- moved D6 26.6 mm to (174.9, 71.3), turned to -45 degrees
Routing:
- net GND: track 0.00 -> 13.3 mm, vias 0 -> 48
- net +3.3V: track 76.2 -> 82.7 mm, vias 9 -> 10
- net /LED4: track 0.00 -> 4.33 mm, vias 0 -> 1
- net /LED1: track 0.00 -> 3.97 mm, vias 0 -> 1
- net /LED3: track 0.00 -> 3.85 mm, vias 0 -> 1
- net /LED2: track 0.00 -> 3.46 mm, vias 0 -> 1
- net /LED 4: track 0.00 -> 2.19 mm
- net /LED 1: track 0.00 -> 2.13 mm
- net /LED 3: track 0.00 -> 1.86 mm
- net /LED 2: track 0.00 -> 1.76 mm
